Commit message: update launch files

File: multi_fetch_gazebo/urdf/kinect_camera.xacro (robot description, xacro)
@@ -1,86 +1,86 @@
 <?xml version="1.0"?>
 <robot name="kinect_camera" xmlns:xacro="http://ros.org/wiki/xacro">
-    <xacro:property name="idx" value="$(arg idx)"/>
-    <!-- base_link -->
-    <link name="kinect_camera_$(arg idx)">
-        <inertial>
-            <origin xyz="0 0 0" rpy="0 0 0"/>
-            <mass value="0.001"/>
-            <inertia ixx="0"  ixy="0"  ixz="0" iyy="0" iyz="0" izz="0" />
-        </inertial>
-        <visual>
-            <origin xyz="0 0 0"/>
-            <geometry>
-                <mesh filename="package://multi_robot_gazebo/meshes/kinect.dae"/>
-            </geometry>
-        </visual>
-        <collision>
-            <origin xyz="0 0 0"/>
-            <geometry>
-                <box size="0.001 0.001 0.001" />
-            </geometry>
-        </collision>
-    </link>
-    <!-- disable gravity -->
-    <gazebo reference="kinect_camera_$(arg idx)">
-        <gravity>false</gravity>
-    </gazebo>
-    <!-- camera sensor in base_link -->
-    <gazebo reference="kinect_camera_$(arg idx)">
-        <!-- origin xyz="0 0 0" rpy="0 0 0"/ -->
-        <sensor type="depth" name="camera">
-            <!--origin xyz="0 0 0" rpy="0 0 0"/ -->
-            <always_on>true</always_on>
-            <update_rate>100</update_rate>
-            <camera>
-                <horizontal_fov>1.047198</horizontal_fov>
-                <image>
-                    <format>R8G8B8</format>
-                    <width>640</width>
-                    <height>480</height>
-                </image>
-                <clip>
-                    <near>0.05</near>
-                    <far>3</far>
-                </clip>
-            </camera>
-            <plugin name="kinect_camera_controller" filename="libgazebo_ros_openni_kinect.so">
-                <!--xacro:property name="cam_name" value="wtf" /-->
-                <baseline>0.2</baseline>
-                <alwaysOn>true</alwaysOn>
-                <updateRate>0.0</updateRate>
-                <cameraName>kinect_camera_$(arg idx)</cameraName>
-                <imageTopicName>rgb/image_raw</imageTopicName>
-                <depthImageTopicName>depth/image_raw</depthImageTopicName>
-                <pointCloudTopicName>depth/points</pointCloudTopicName>
-                <cameraInfoTopicName>rgb/camera_info</cameraInfoTopicName>
-                <depthImageCameraInfoTopicName>depth/camera_info</depthImageCameraInfoTopicName>
-                <frameName>kinect_camera_frame_$(arg idx)</frameName>
-                <pointCloudCutoff>0.0001</pointCloudCutoff>
-                <pointCloudCutoffMax>3.0</pointCloudCutoffMax>
-                <distortionK1>0</distortionK1>
-                <distortionK2>0</distortionK2>
-                <distortionK3>0</distortionK3>
-                <distortionT1>0</distortionT1>
-                <distortionT2>0</distortionT2>
-                <CxPrime>0</CxPrime>
-                <Cx>0</Cx>
-                <Cy>0</Cy>
-                <focalLength>0</focalLength>
-                <hackBaseline>0</hackBaseline>
-            </plugin>
-        </sensor>
-    </gazebo>
-    <gazebo>
-        <plugin name="p3d_base_controller" filename="libgazebo_ros_p3d.so">
+  <xacro:property name="idx" value="$(arg idx)"/>
+  <!-- base_link -->
+  <link name="base_link">
+    <inertial>
+      <origin xyz="0 0 0" rpy="0 0 0"/>
+      <mass value="0.001"/>
+      <inertia ixx="0"  ixy="0"  ixz="0" iyy="0" iyz="0" izz="0" />
+    </inertial>
+    <!-- <visual> -->
+      <!-- <origin xyz="0 0 0"/> -->
+      <!-- <geometry> -->
+          <!-- <mesh filename="package://multi_fetch_gazebo/meshes/kinect.dae"/> -->
+      <!-- </geometry> -->
+    <!-- </visual> -->
+    <collision>
+      <origin xyz="0 0 0"/>
+      <geometry>
+          <box size="0.001 0.001 0.001" />
+      </geometry>
+    </collision>
+  </link>
+  <!-- disable gravity -->
+  <gazebo reference="base_link">
+    <gravity>false</gravity>
+  </gazebo>
+  <!-- camera sensor in base_link -->
+  <gazebo reference="base_link">
+    <!-- origin xyz="0 0 0" rpy="0 0 0"/ -->
+    <sensor type="depth" name="camera">
+      <!--origin xyz="0 0 0" rpy="0 0 0"/ -->
+      <always_on>true</always_on>
+      <update_rate>15.0</update_rate>
+      <camera>
+        <horizontal_fov>1.047197</horizontal_fov>
+        <image>
+          <format>R8G8B8</format>
+          <width>640</width>
+          <height>480</height>
+        </image>
+        <clip>
+          <near>0.05</near>
+          <far>50</far>
+        </clip>
+      </camera>
+      <plugin name="kinect_camera_controller" filename="libgazebo_ros_openni_kinect.so">
+        <!--xacro:property name="cam_name" value="wtf" /-->
+        <baseline>0.1</baseline>
         <alwaysOn>true</alwaysOn>
-        <updateRate>100</updateRate>
-        <bodyName>kinect_camera_$(arg idx)</bodyName>
-        <topicName>kinect_camera_$(arg idx)_ground_truth</topicName>
-        <gaussianNoise>0</gaussianNoise>
-        <frameName>map</frameName>
-        <xyzOffsets>0 0 0</xyzOffsets>
-        <rpyOffsets>0 0 0</rpyOffsets>
-        </plugin>
-    </gazebo>
+        <updateRate>1000</updateRate>
+        <cameraName>main_camera</cameraName>
+        <imageTopicName>rgb/image_raw</imageTopicName>
+        <depthImageTopicName>depth/image_raw</depthImageTopicName>
+        <pointCloudTopicName>depth/points</pointCloudTopicName>
+        <cameraInfoTopicName>rgb/camera_info</cameraInfoTopicName>
+        <depthImageCameraInfoTopicName>depth/camera_info</depthImageCameraInfoTopicName>
+        <frameName>kinect_camera_$(arg idx)/robot_camera_frame</frameName>
+        <pointCloudCutoff>0.35</pointCloudCutoff>
+        <pointCloudCutoffMax>3.0</pointCloudCutoffMax>
+        <distortionK1>0</distortionK1>
+        <distortionK2>0</distortionK2>
+        <distortionK3>0</distortionK3>
+        <distortionT1>0</distortionT1>
+        <distortionT2>0</distortionT2>
+        <CxPrime>0</CxPrime>
+        <Cx>0</Cx>
+        <Cy>0</Cy>
+        <focalLength>0</focalLength>
+        <hackBaseline>0</hackBaseline>
+      </plugin>
+    </sensor>
+  </gazebo>
+  <gazebo>
+    <plugin name="p3d_base_controller" filename="libgazebo_ros_p3d.so">
+    <alwaysOn>true</alwaysOn>
+    <updateRate>1000</updateRate>
+    <bodyName>base_link</bodyName>
+    <topicName>base_link_ground_truth</topicName>
+    <gaussianNoise>0</gaussianNoise>
+    <frameName>map</frameName>
+    <xyzOffsets>0 0 0</xyzOffsets>
+    <rpyOffsets>0 0 0</rpyOffsets>
+    </plugin>
+  </gazebo>
 </robot>
